Commit message: Updated files with recent changes

File: install/robot_description/share/robot_description/urdf/cropMap_urdf.urdf (robot description, URDF)
Before this commit: robot cropMap_urdf, 15 links, 14 joints
Links:
- added link back_camera_optical_frame
- added link front_camera_optical_frame
Joints:
- added joint back_camera_optical_joint: type fixed, parent back_camera, child back_camera_optical_frame, origin xyz=0 0 0 rpy=-1.5708 0 1.5708
- added joint front_camera_optical_joint: type fixed, parent front_camera, child front_camera_optical_frame, origin xyz=0 0 0 rpy=-1.5708 0 -1.5708

File: install/robot_description/share/robot_description/urdf/robot.urdf.xacro (robot description, xacro)
@@ -21,4 +21,7 @@
     <color rgba="0.0 0.0 0.0 1.0"/>
   </material>
+  <material name="red">
+    <color rgba="1.0 0.0 0.0 1.0"/>
+  </material>
   <!-- Base Link -->
   <link name="base_link">
@@ -249,12 +252,73 @@
   </joint>
   <!-- Gazebo plugin for back camera -->
-<gazebo reference="back_camera">
-  <sensor type="camera" name="back_camera">
-    <topic>back_camera</topic>
-    <camera>
+  <gazebo reference="back_camera">
+    <sensor type="camera" name="back_camera">
+      <update_rate>30.0</update_rate>
+      <camera name="back">
+        <horizontal_fov>1.047</horizontal_fov>
+        <image>
+          <width>640</width>
+          <height>480</height>
+          <format>R8G8B8</format>
+        </image>
+        <clip>
+          <near>0.1</near>
+          <far>100</far>
+        </clip>
+        <noise>
+          <type>gaussian</type>
+          <mean>0.0</mean>
+          <stddev>0.007</stddev>
+        </noise>
+      </camera>
+      <plugin name="back_camera_controller" filename="libgazebo_ros_camera.so">
+        <alwaysOn>true</alwaysOn>
+        <updateRate>0.0</updateRate>
+        <cameraName>back_camera</cameraName>
+        <imageTopicName>image_raw</imageTopicName>
+        <cameraInfoTopicName>camera_info</cameraInfoTopicName>
+        <frameName>back_camera_optical_frame</frameName>
+        <hackBaseline>0.07</hackBaseline>
+        <distortionK1>0.0</distortionK1>
+        <distortionK2>0.0</distortionK2>
+        <distortionK3>0.0</distortionK3>
+        <distortionT1>0.0</distortionT1>
+        <distortionT2>0.0</distortionT2>
+      </plugin>
+    </sensor>
+  </gazebo>
+  <!-- Front Camera -->
+  <link name="front_camera">
+    <inertial>
+      <origin xyz="0.012395 -0.012586 0.0091516" rpy="0 0 0" />
+      <mass value="0.1" />
+      <inertia
+        ixx="0.001" ixy="0.0" ixz="0.0"
+        iyy="0.001" iyz="0.0"
+        izz="0.001" />
+    </inertial>
+    <visual>
+      <origin xyz="0 0 0" rpy="0 0 0" />
+      <geometry>
+        <mesh filename="file:///home/student/eiratech_ws/src/robot_description/meshes/front_camera.STL" />
+      </geometry>
+      <material name="black"/>
+    </visual>
+  </link>
+  <joint name="front_camera_joint" type="fixed">
+    <origin xyz="0.42423 0.0126 0.060602" rpy="0 0 0" />
+    <parent link="base_link" />
+    <child link="front_camera" />
+  </joint>
+  <!-- Gazebo plugin for front camera -->
+  <gazebo reference="front_camera">
+  <sensor type="camera" name="front_camera">
+    <update_rate>30.0</update_rate>
+    <camera name="front">
       <horizontal_fov>1.047</horizontal_fov>
       <image>
         <width>640</width>
         <height>480</height>
+        <format>R8G8B8</format>
       </image>
       <clip>
@@ -262,52 +326,13 @@
         <far>100</far>
       </clip>
+      <noise>
+        <type>gaussian</type>
+        <mean>0.0</mean>
+        <stddev>0.007</stddev>
+      </noise>
     </camera>
-    <plugin filename="libgz_sim_camera_system.so" name="gz_sim_camera">
-      <topic>back_camera</topic>
-      <frame_name>back_camera</frame_name>
-    </plugin>
-  </sensor>
-</gazebo>
-  <!-- Front Camera -->
-  <link name="front_camera">
-    <inertial>
-      <origin xyz="0.012395 -0.012586 0.0091516" rpy="0 0 0" />
-      <mass value="0.1" />
-      <inertia
-        ixx="0.001" ixy="0.0" ixz="0.0"
-        iyy="0.001" iyz="0.0"
-        izz="0.001" />
-    </inertial>
-    <visual>
-      <origin xyz="0 0 0" rpy="0 0 0" />
-      <geometry>
-        <mesh filename="file:///home/student/eiratech_ws/src/robot_description/meshes/front_camera.STL" />
-      </geometry>
-      <material name="black"/>
-    </visual>
-  </link>
-  <joint name="front_camera_joint" type="fixed">
-    <origin xyz="0.42423 0.0126 0.060602" rpy="0 0 0" />
-    <parent link="base_link" />
-    <child link="front_camera" />
-  </joint>
-  <!-- Gazebo plugin for front camera -->
-<gazebo reference="front_camera">
-  <sensor type="camera" name="front_camera">
-    <topic>front_camera</topic>
-    <camera>
-      <horizontal_fov>1.047</horizontal_fov>
-      <image>
-        <width>640</width>
-        <height>480</height>
-      </image>
-      <clip>
-        <near>0.1</near>
-        <far>100</far>
-      </clip>
-    </camera>
-    <plugin filename="libgz_sim_camera_system.so" name="gz_sim_camera">
-      <topic>front_camera</topic>
-      <frame_name>front_camera</frame_name>
+    <plugin filename="gz-sim-sensors-system" name="gz::sim::systems::Sensors">
+      <render_engine>ogre2</render_engine>
+      <topic>/front_camera</topic>
     </plugin>
   </sensor>
@@ -353,4 +378,10 @@
     <axis xyz="1 0 0" />
   </joint>
+  <link name="front_camera_optical_frame"/>
+  <joint name="front_camera_optical_joint" type="fixed">
+    <origin xyz="0 0 0" rpy="-1.5708 0 -1.5708" />
+    <parent link="front_camera" />
+    <child link="front_camera_optical_frame" />
+  </joint>
   <link name="back_camera_dummy"/>
   <joint name="back_camera_dummy_joint" type="fixed">
@@ -359,4 +390,10 @@
     <child link="back_camera_dummy" />
     <axis xyz="1 0 0" />
+  </joint>
+  <link name="back_camera_optical_frame"/>
+  <joint name="back_camera_optical_joint" type="fixed">
+    <origin xyz="0 0 0" rpy="-1.5708 0 1.5708" />
+    <parent link="back_camera" />
+    <child link="back_camera_optical_frame" />
   </joint>
    <!-- Add RGB-D Sensor -->
@@ -475,48 +512,44 @@
   <!-- Gazebo plugin for LiDAR -->
   <gazebo reference="lidar_link">
-    <material>Gazebo/Black</material>
-    <sensor type="ray" name="lidar_sensor">
-      <pose>0 0 0 0 0 0</pose>
-      <visualize>true</visualize>
-      <update_rate>10</update_rate>
-      <ray>
-        <scan>
-          <horizontal>
-            <samples>360</samples>
-            <resolution>1</resolution>
-            <min_angle>-3.14159</min_angle>
-            <max_angle>3.14159</max_angle>
-          </horizontal>
-        </scan>
-        <range>
-          <min>0.1</min>
-          <max>30.0</max>
-          <resolution>0.01</resolution>
-        </range>
-        <noise>
-          <type>gaussian</type>
-          <mean>0.0</mean>
-          <stddev>0.01</stddev>
-        </noise>
-      </ray>
-      <plugin name="lidar_controller" filename="libgazebo_ros_ray_sensor.so">
-        <ros>
-          <namespace>/cropMap</namespace>
-          <remapping>~/out:=scan</remapping>
-        </ros>
-        <output_type>sensor_msgs/LaserScan</output_type>
-        <frame_name>lidar_link</frame_name>
-      </plugin>
-    </sensor>
-  </gazebo>
+  <sensor type="gpu_lidar" name="lidar_sensor">
+    <pose>0 0 0 0 0 0</pose>
+    <visualize>true</visualize>
+    <update_rate>10</update_rate>
+    <lidar>
+      <scan>
+        <horizontal>
+          <samples>360</samples>
+          <resolution>1</resolution>
+          <min_angle>-3.14159</min_angle>
+          <max_angle>3.14159</max_angle>
+        </horizontal>
+      </scan>
+      <range>
+        <min>0.1</min>
+        <max>30.0</max>
+        <resolution>0.01</resolution>
+      </range>
+      <noise>
+        <type>gaussian</type>
+        <mean>0.0</mean>
+        <stddev>0.01</stddev>
+      </noise>
+    </lidar>
+    <plugin filename="gz-sim-sensors-system" name="gz::sim::systems::Sensors">
+      <topic>/lidar</topic>
+    </plugin>
+  </sensor>
+</gazebo>
   <!-- Skid Steering Drive Controller -->
   <gazebo>
-  <plugin filename="libgz_sim_diff_drive_system.so" name="gz_sim_diff_drive">
+  <plugin filename="gz-sim-diff-drive-system" name="gz::sim::systems::DiffDrive">
     <left_joint>wheel_front_left_joint</left_joint>
     <left_joint>wheel_back_left_joint</left_joint>
     <right_joint>wheel_front_right_joint</right_joint>
     <right_joint>wheel_back_right_joint</right_joint>
-    <wheel_separation>0.4</wheel_separation>
+    <wheel_separation>0.56</wheel_separation>
     <wheel_radius>0.1</wheel_radius>
+    <topic>cmd_vel</topic>
+    <odom_topic>odom</odom_topic>
     <odom_publish_frequency>50</odom_publish_frequency>
     <max_linear_acceleration>1.0</max_linear_acceleration>
@@ -528,11 +561,7 @@
     <max_angular_velocity>1.0</max_angular_velocity>
     <min_angular_velocity>-1.0</min_angular_velocity>
-    <topic>cmd_vel</topic>
-    <odom_topic>odom</odom_topic>
-    <odom_frame>odom</odom_frame>
-    <robot_base_frame>base_link</robot_base_frame>
   </plugin>
 </gazebo>
-  <!-- IMU Sensor -->
+   <!-- IMU Sensor -->
   <link name="imu_link">
     <inertial>
@@ -560,24 +589,14 @@
     <origin xyz="0 0 0.1" rpy="0 0 0"/>
   </joint>
+  <!--IMU plugin -->
   <gazebo reference="imu_link">
-    <material>Gazebo/Blue</material>
-    <gravity>true</gravity>
-    <sensor name="imu_sensor" type="imu">
-      <always_on>true</always_on>
-      <update_rate>100</update_rate>
-      <visualize>true</visualize>
-      <topic>__default_topic__</topic>
-      <plugin filename="libgazebo_ros_imu_sensor.so" name="imu_plugin">
-        <topicName>imu</topicName>
-        <bodyName>imu_link</bodyName>
-        <updateRateHZ>100.0</updateRateHZ>
-        <gaussianNoise>0.0</gaussianNoise>
-        <xyzOffset>0 0 0</xyzOffset>
-        <rpyOffset>0 0 0</rpyOffset>
-        <frameName>imu_link</frameName>
-        <initialOrientationAsReference>false</initialOrientationAsReference>
-      </plugin>
-      <pose>0 0 0 0 0 0</pose>
-    </sensor>
-  </gazebo>
+  <sensor type="imu" name="imu_sensor">
+    <always_on>true</always_on>
+    <update_rate>100</update_rate>
+    <visualize>true</visualize>
+    <plugin filename="gz-sim-imu-system" name="gz::sim::systems::Imu">
+      <topic>/imu</topic>
+    </plugin>
+  </sensor>
+ </gazebo>
 </robot>

Commit message: Initial commit

File: install/robot_description/share/robot_description/urdf/cropMap_urdf.urdf (robot description, URDF)
Before this commit: robot cropMap_urdf, 17 links, 16 joints
Links:
- removed link back_camera_dummy
- removed link front_camera_dummy
- link TC_V0: geometry collision mesh filename=package://robot_description/meshes/TC_V0.STL; visual mesh filename=package://robot_description/meshes/TC_V0.STL
- link back_camera: geometry visual mesh filename=package://robot_description/meshes/back_camera.STL
- link base_footprint: mass None -> 0.1
- link base_link: geometry collision mesh filename=package://robot_description/meshes/base_link.STL; visual mesh filename=package://robot_description/meshes/base_link.STL
- link front_camera: geometry visual mesh filename=package://robot_description/meshes/front_camera.STL
- link wheel_back_left: geometry collision mesh filename=package://robot_description/meshes/wheel_back_left.STL; visual mesh filename=package://robot_description/meshes/wheel_back_left.STL
- link wheel_back_right: geometry collision mesh filename=package://robot_description/meshes/wheel_back_right.STL; visual mesh filename=package://robot_description/meshes/wheel_back_right.STL
- link wheel_front_left: geometry collision mesh filename=package://robot_description/meshes/wheel_front_left.STL; visual mesh filename=package://robot_description/meshes/wheel_front_left.STL
- link wheel_front_right: geometry collision mesh filename=package://robot_description/meshes/wheel_front_right.STL; visual mesh filename=package://robot_description/meshes/wheel_front_right.STL
Joints:
- removed joint back_camera_dummy_joint
- removed joint front_camera_dummy_joint
