Commit message: Nav2 intergration

File: install/robot_description/share/robot_description/urdf/robot.urdf.xacro (robot description, xacro)
@@ -1,602 +1 @@
-<?xml version="1.0" ?>
-<robot name="cropMap_urdf" xmlns:xacro="http://www.ros.org/wiki/xacro">
-  <!-- Gazebo plugin includes -->
-  <gazebo>
-    <plugin name="gazebo_ros_control" filename="libgazebo_ros_control.so">
-      <robotNamespace>/cropMap_urdf</robotNamespace>
-      <robotSimType>gazebo_ros_control/DefaultRobotHWSim</robotSimType>
-    </plugin>
-  </gazebo>
-  <!-- Include Gazebo colors -->
-  <material name="dark_grey">
-    <color rgba="0.3 0.3 0.3 1.0"/>
-  </material>
-  <material name="light_grey">
-    <color rgba="0.79216 0.81961 0.93333 1"/>
-  </material>
-  <material name="blue">
-    <color rgba="0.0 0.0 0.8 1.0"/>
-  </material>
-  <material name="black">
-    <color rgba="0.0 0.0 0.0 1.0"/>
-  </material>
-  <material name="red">
-    <color rgba="1.0 0.0 0.0 1.0"/>
-  </material>
-  <!-- Base Link -->
-  <link name="base_link">
-    <inertial>
-      <origin xyz="0.018582 -0.00058815 -0.099852" rpy="0 0 0" />
-      <mass value="32.31" />
-      <inertia
-        ixx="0.92" ixy="0" ixz="0"
-        iyy="3.12" iyz="0"
-        izz="2.87" />
-    </inertial>
-    <visual>
-      <origin xyz="0 0 0" rpy="0 0 0" />
-      <geometry>
-        <mesh filename="file:///home/student/eiratech_ws/src/robot_description/meshes/base_link.STL" />
-      </geometry>
-      <material name="light_grey"/>
-    </visual>
-    <collision>
-      <origin xyz="0 0 0" rpy="0 0 0" />
-      <geometry>
-        <mesh filename="file:///home/student/eiratech_ws/src/robot_description/meshes/base_link.STL" />
-      </geometry>
-    </collision>
-  </link>
-  <!-- Gazebo material for base_link -->
-  <gazebo reference="base_link">
-    <material>Gazebo/Gray</material>
-  </gazebo>
-  <!-- Base footprint -->
-  <link name="base_footprint"/>
-  <joint name="base_footprint_ref_joint" type="fixed">
-    <origin xyz="0 0 .25" rpy="0 0 0" />
-    <parent link="base_footprint" />
-    <child link="base_link" />
-    <axis xyz="0 1 0" />
-  </joint>
-  <!-- Front Right Wheel -->
-  <link name="wheel_front_right">
-    <inertial>
-      <origin xyz="-3.8916E-11 0.012822 1.02E-07" rpy="0 0 0" />
-      <mass value=".041" />
-      <inertia
-        ixx="0.04" ixy="0.0" ixz="0.0"
-        iyy="0.05" iyz="0.0"
-        izz="0.04" />
-    </inertial>
-    <visual>
-      <origin xyz="0 0 0" rpy="0 0 0" />
-      <geometry>
-        <mesh filename="file:///home/student/eiratech_ws/src/robot_description/meshes/wheel_front_right.STL" />
-      </geometry>
-      <material name="light_grey"/>
-    </visual>
-    <collision>
-      <origin xyz="0 0 0" rpy="0 0 0" />
-      <geometry>
-        <mesh filename="file:///home/student/eiratech_ws/src/robot_description/meshes/wheel_front_right.STL" />
-      </geometry>
-    </collision>
-  </link>
-  <joint name="wheel_front_right_joint" type="continuous">
-    <origin xyz="0.37976 0.2802 -0.078259" rpy="0 0 0" />
-    <parent link="base_link" />
-    <child link="wheel_front_right" />
-    <axis xyz="0 1 0" />
-    <dynamics damping="0.0001" friction="0.0001" />
-  </joint>
-  <!-- Gazebo plugin for front right wheel -->
-  <gazebo reference="wheel_front_right">
-    <material>Gazebo/DarkGray</material>
-    <mu1>1.0</mu1>
-    <mu2>1.0</mu2>
-    <kp>1000000.0</kp>
-    <kd>100.0</kd>
-    <minDepth>0.001</minDepth>
-    <maxVel>1.0</maxVel>
-    <fdir1>1 0 0</fdir1>
-  </gazebo>
-  <!-- Back Right Wheel -->
-  <link name="wheel_back_right">
-    <inertial>
-      <origin xyz="-3.8916E-11 0.012822 1.02E-07" rpy="0 0 0" />
-      <mass value=".041" />
-      <inertia
-        ixx="0.04" ixy="0.0" ixz="0.0"
-        iyy="0.05" iyz="0.0"
-        izz="0.04" />
-    </inertial>
-    <visual>
-      <origin xyz="0 0 0" rpy="0 0 0" />
-      <geometry>
-        <mesh filename="file:///home/student/eiratech_ws/src/robot_description/meshes/wheel_back_right.STL" />
-      </geometry>
-      <material name="light_grey"/>
-    </visual>
-    <collision>
-      <origin xyz="0 0 0" rpy="0 0 0" />
-      <geometry>
-        <mesh filename="file:///home/student/eiratech_ws/src/robot_description/meshes/wheel_back_right.STL" />
-      </geometry>
-    </collision>
-  </link>
-  <joint name="wheel_back_right_joint" type="continuous">
-    <origin xyz="-0.38026 0.2802 -0.078259" rpy="0 0 0" />
-    <parent link="base_link" />
-    <child link="wheel_back_right" />
-    <axis xyz="0 1 0" />
-    <dynamics damping="0.0001" friction="0.0001" />
-  </joint>
-  <!-- Gazebo plugin for back right wheel -->
-  <gazebo reference="wheel_back_right">
-    <material>Gazebo/DarkGray</material>
-    <mu1>1.0</mu1>
-    <mu2>1.0</mu2>
-    <kp>1000000.0</kp>
-    <kd>100.0</kd>
-    <minDepth>0.001</minDepth>
-    <maxVel>1.0</maxVel>
-    <fdir1>1 0 0</fdir1>
-  </gazebo>
-  <!-- Back Left Wheel -->
-  <link name="wheel_back_left">
-    <inertial>
-      <origin xyz="-1.02E-07 -0.012822 3.8916E-11" rpy="0 0 0" />
-      <mass value=".041" />
-      <inertia
-        ixx="0.04" ixy="0.0" ixz="0.0"
-        iyy="0.05" iyz="0.0"
-        izz="0.04" />
-    </inertial>
-    <visual>
-      <origin xyz="0 0 0" rpy="0 0 0" />
-      <geometry>
-        <mesh filename="file:///home/student/eiratech_ws/src/robot_description/meshes/wheel_back_left.STL" />
-      </geometry>
-      <material name="light_grey"/>
-    </visual>
-    <collision>
-      <origin xyz="0 0 0" rpy="0 0 0" />
-      <geometry>
-        <mesh filename="file:///home/student/eiratech_ws/src/robot_description/meshes/wheel_back_left.STL" />
-      </geometry>
-    </collision>
-  </link>
-  <joint name="wheel_back_left_joint" type="continuous">
-    <origin xyz="-0.38026 -0.2802 -0.078259" rpy="0 0 0" />
-    <parent link="base_link" />
-    <child link="wheel_back_left" />
-    <axis xyz="0 1 0" />
-    <dynamics damping="0.0001" friction="0.0001" />
-  </joint>
-  <!-- Gazebo plugin for back left wheel -->
-  <gazebo reference="wheel_back_left">
-    <material>Gazebo/DarkGray</material>
-    <mu1>1.0</mu1>
-    <mu2>1.0</mu2>
-    <kp>1000000.0</kp>
-    <kd>100.0</kd>
-    <minDepth>0.001</minDepth>
-    <maxVel>1.0</maxVel>
-    <fdir1>1 0 0</fdir1>
-  </gazebo>
-  <!-- Front Left Wheel -->
-  <link name="wheel_front_left">
-    <inertial>
-      <origin xyz="3.8916E-11 -0.012822 1.02E-07" rpy="0 0 0" />
-      <mass value=".041" />
-      <inertia
-        ixx="0.04" ixy="0.0" ixz="0.0"
-        iyy="0.05" iyz="0.0"
-        izz="0.04" />
-    </inertial>
-    <visual>
-      <origin xyz="0 0 0" rpy="0 0 0" />
-      <geometry>
-        <mesh filename="file:///home/student/eiratech_ws/src/robot_description/meshes/wheel_front_left.STL" />
-      </geometry>
-      <material name="light_grey"/>
-    </visual>
-    <collision>
-      <origin xyz="0 0 0" rpy="0 0 0" />
-      <geometry>
-        <mesh filename="file:///home/student/eiratech_ws/src/robot_description/meshes/wheel_front_left.STL" />
-      </geometry>
-    </collision>
-  </link>
-  <joint name="wheel_front_left_joint" type="continuous">
-    <origin xyz="0.37976 -0.2802 -0.078259" rpy="0 0 0" />
-    <parent link="base_link" />
-    <child link="wheel_front_left" />
-    <axis xyz="0 1 0" />
-    <dynamics damping="0.0001" friction="0.0001" />
-  </joint>
-  <!-- Gazebo plugin for front left wheel -->
-  <gazebo reference="wheel_front_left">
-    <material>Gazebo/DarkGray</material>
-    <mu1>1.0</mu1>
-    <mu2>1.0</mu2>
-    <kp>1000000.0</kp>
-    <kd>100.0</kd>
-    <minDepth>0.001</minDepth>
-    <maxVel>1.0</maxVel>
-    <fdir1>1 0 0</fdir1>
-  </gazebo>
-  <!-- Back Camera -->
-  <link name="back_camera">
-    <inertial>
-      <origin xyz="-0.032487 0.0089676 -0.0027971" rpy="0 0 0" />
-      <mass value="0.1" />
-      <inertia
-        ixx="0.001" ixy="0.0" ixz="0.0"
-        iyy="0.001" iyz="0.0"
-	      izz="0.001" />
-    </inertial>
-    <visual>
-      <origin xyz="0 0 0" rpy="0 0 0" />
-      <geometry>
-        <mesh filename="file:///home/student/eiratech_ws/src/robot_description/meshes/back_camera.STL" />
-      </geometry>
-      <material name="black"/>
-    </visual>
-  </link>
-  <joint name="back_camera_joint" type="fixed">
-    <origin xyz="-0.40479 -0.0089685 0.073466" rpy="0 0 0" />
-    <parent link="base_link" />
-    <child link="back_camera" />
-  </joint>
-  <!-- Gazebo plugin for back camera -->
-  <gazebo reference="back_camera">
-    <sensor type="camera" name="back_camera">
-      <update_rate>30.0</update_rate>
-      <camera name="back">
-        <horizontal_fov>1.047</horizontal_fov>
-        <image>
-          <width>640</width>
-          <height>480</height>
-          <format>R8G8B8</format>
-        </image>
-        <clip>
-          <near>0.1</near>
-          <far>100</far>
-        </clip>
-        <noise>
-          <type>gaussian</type>
-          <mean>0.0</mean>
-          <stddev>0.007</stddev>
-        </noise>
-      </camera>
-      <plugin name="back_camera_controller" filename="libgazebo_ros_camera.so">
-        <alwaysOn>true</alwaysOn>
-        <updateRate>0.0</updateRate>
-        <cameraName>back_camera</cameraName>
-        <imageTopicName>image_raw</imageTopicName>
-        <cameraInfoTopicName>camera_info</cameraInfoTopicName>
-        <frameName>back_camera_optical_frame</frameName>
-        <hackBaseline>0.07</hackBaseline>
-        <distortionK1>0.0</distortionK1>
-        <distortionK2>0.0</distortionK2>
-        <distortionK3>0.0</distortionK3>
-        <distortionT1>0.0</distortionT1>
-        <distortionT2>0.0</distortionT2>
-      </plugin>
-    </sensor>
-  </gazebo>
-  <!-- Front Camera -->
-  <link name="front_camera">
-    <inertial>
-      <origin xyz="0.012395 -0.012586 0.0091516" rpy="0 0 0" />
-      <mass value="0.1" />
-      <inertia
-        ixx="0.001" ixy="0.0" ixz="0.0"
-        iyy="0.001" iyz="0.0"
-        izz="0.001" />
-    </inertial>
-    <visual>
-      <origin xyz="0 0 0" rpy="0 0 0" />
-      <geometry>
-        <mesh filename="file:///home/student/eiratech_ws/src/robot_description/meshes/front_camera.STL" />
-      </geometry>
-      <material name="black"/>
-    </visual>
-  </link>
-  <joint name="front_camera_joint" type="fixed">
-    <origin xyz="0.42423 0.0126 0.060602" rpy="0 0 0" />
-    <parent link="base_link" />
-    <child link="front_camera" />
-  </joint>
-  <!-- Gazebo plugin for front camera -->
-  <gazebo reference="front_camera">
-  <sensor type="camera" name="front_camera">
-    <update_rate>30.0</update_rate>
-    <camera name="front">
-      <horizontal_fov>1.047</horizontal_fov>
-      <image>
-        <width>640</width>
-        <height>480</height>
-        <format>R8G8B8</format>
-      </image>
-      <clip>
-        <near>0.1</near>
-        <far>100</far>
-      </clip>
-      <noise>
-        <type>gaussian</type>
-        <mean>0.0</mean>
-        <stddev>0.007</stddev>
-      </noise>
-    </camera>
-    <plugin filename="gz-sim-sensors-system" name="gz::sim::systems::Sensors">
-      <render_engine>ogre2</render_engine>
-      <topic>/front_camera</topic>
-    </plugin>
-  </sensor>
-</gazebo>
-  <!-- TC_V0 -->
-  <link name="TC_V0">
-    <inertial>
-      <origin xyz="-7.5077E-05 -2.3538E-06 -0.015092" rpy="0 0 0" />
-      <mass value="14.01" />
-      <inertia
-        ixx="0.66" ixy="0.0" ixz="0.0"
-        iyy="1.01" iyz="0.0"
-        izz="1.66" />
-    </inertial>
-    <visual>
-      <origin xyz="0 0 0" rpy="0 0 0" />
-      <geometry>
-        <mesh filename="file:///home/student/eiratech_ws/src/robot_description/meshes/TC_V0.STL" />
-      </geometry>
-      <material name="light_grey"/>
-    </visual>
-    <collision>
-      <origin xyz="0 0 0" rpy="0 0 0" />
-      <geometry>
-        <mesh filename="file:///home/student/eiratech_ws/src/robot_description/meshes/TC_V0.STL" />
-      </geometry>
-    </collision>
-  </link>
-  <joint name="TC_V0_joint" type="fixed">
-    <origin xyz="0 0 0.16825" rpy="0 0 0" />
-    <parent link="base_link" />
-    <child link="TC_V0" />
-  </joint>
-  <gazebo reference="TC_V0">
-    <material>Gazebo/Gray</material>
-  </gazebo>
-  <!-- Camera dummy frames -->
-  <link name="front_camera_dummy"/>
-  <joint name="front_camera_dummy_joint" type="fixed">
-    <origin xyz="0 0 0" rpy="-1.5708 0 -1.5708" />
-    <parent link="front_camera" />
-    <child link="front_camera_dummy" />
-    <axis xyz="1 0 0" />
-  </joint>
-  <link name="front_camera_optical_frame"/>
-  <joint name="front_camera_optical_joint" type="fixed">
-    <origin xyz="0 0 0" rpy="-1.5708 0 -1.5708" />
-    <parent link="front_camera" />
-    <child link="front_camera_optical_frame" />
-  </joint>
-  <link name="back_camera_dummy"/>
-  <joint name="back_camera_dummy_joint" type="fixed">
-    <origin xyz="0 0 0" rpy="-1.5708 0 1.5708" />
-    <parent link="back_camera" />
-    <child link="back_camera_dummy" />
-    <axis xyz="1 0 0" />
-  </joint>
-  <link name="back_camera_optical_frame"/>
-  <joint name="back_camera_optical_joint" type="fixed">
-    <origin xyz="0 0 0" rpy="-1.5708 0 1.5708" />
-    <parent link="back_camera" />
-    <child link="back_camera_optical_frame" />
-  </joint>
-   <!-- Add RGB-D Sensor -->
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
File: src/robot_description/urdf/cropMap_urdf.urdf (robot description, URDF)
Before this commit: robot cropMap_urdf, 15 links, 14 joints
Links:
- removed link back_camera_optical_frame
- removed link front_camera_optical_frame
- removed link rgbd_camera_link
- removed link rgbd_camera_optical_frame
- added link back_camera_dummy
- added link front_camera_dummy
- added link gps_link, mass 0.05; collision cylinder length=0.1 radius=0.02; visual cylinder length=0.1 radius=0.02
- link TC_V0: geometry collision mesh filename=file:///home/manish/eiratech_ws/install/robot_description/s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; visual mesh filename=file:///home/manish/eiratech_ws/install/robot_description/s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
- link back_camera: mass 0.1 -> 0.2; geometry visual mesh filename=file:///home/manish/eiratech_ws/install/robot_description/s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
- link base_footprint: mass 0.1 -> None
- link base_link: geometry collision mesh filename=file:///home/manish/eiratech_ws/install/robot_description/s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; visual mesh filename=file:///home/manish/eiratech_ws/install/robot_description/s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
- link front_camera: mass 0.1 -> 0.2; geometry visual mesh filename=file:///home/manish/eiratech_ws/install/robot_description/s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
- link imu_link: mass 0.01 -> 0.1; geometry collision box size=0.05 0.05 0.02; visual box size=0.05 0.05 0.02
- link lidar_link: mass 0.1 -> 0.8; geometry collision cylinder length=0.08 radius=0.05; visual cylinder length=0.08 radius=0.05
- link wheel_back_left: mass .041 -> 2.5; geometry collision mesh filename=file:///home/manish/eiratech_ws/install/robot_description/s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; visual mesh filename=file:///home/manish/eiratech_ws/install/robot_description/s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
- link wheel_back_right: mass .041 -> 2.5; geometry collision mesh filename=file:///home/manish/eiratech_ws/install/robot_description/s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; visual mesh filename=file:///home/manish/eiratech_ws/install/robot_description/s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
- link wheel_front_left: mass .041 -> 2.5; geometry collision mesh filename=file:///home/manish/eiratech_ws/install/robot_description/s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; visual mesh filename=file:///home/manish/eiratech_ws/install/robot_description/s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
- link wheel_front_right: mass .041 -> 2.5; geometry collision mesh filename=file:///home/manish/eiratech_ws/install/robot_description/s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; visual mesh filename=file:///home/manish/eiratech_ws/install/robot_description/s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
Joints:
- removed joint back_camera_optical_joint
- removed joint front_camera_optical_joint
- removed joint rgbd_camera_joint
- removed joint rgbd_camera_optical_joint
- added joint back_camera_dummy_joint: type fixed, parent back_camera, child back_camera_dummy, origin xyz=0 0 0 rpy=-1.5708 0 1.5708, axis 1 0 0
- added joint front_camera_dummy_joint: type fixed, parent front_camera, child front_camera_dummy, origin xyz=0 0 0 rpy=-1.5708 0 -1.5708, axis 1 0 0
- added joint gps_joint: type fixed, parent TC_V0, child gps_link, origin xyz=-0.2 0 0.5 rpy=0 0 0
- joint TC_V0_joint: axis (none) -> 0 0 0
- joint back_camera_joint: axis (none) -> 0 0 0
- joint front_camera_joint: axis (none) -> 0 0 0
- joint lidar_joint: origin xyz=0 0 0.25 rpy=0 0 0 -> xyz=0 0 0.4 rpy=0 0 0

File: src/robot_description/urdf/dummy.urdf (robot description, URDF)
Before this commit: robot cropMap_urdf, 15 links, 14 joints
Links:
- removed link back_camera_dummy
- removed link front_camera_dummy
- added link back_camera_optical_frame
- added link front_camera_optical_frame
- link TC_V0: geometry collision mesh filename=package://robot_description/meshes/TC_V0.STL; visual mesh filename=package://robot_description/meshes/TC_V0.STL
- link back_camera: geometry visual mesh filename=package://robot_description/meshes/back_camera.STL
- link base_footprint: mass None -> 0.1
- link base_link: geometry collision mesh filename=package://robot_description/meshes/base_link.STL; visual mesh filename=package://robot_description/meshes/base_link.STL
- link front_camera: geometry visual mesh filename=package://robot_description/meshes/front_camera.STL
- link wheel_back_left: geometry collision mesh filename=package://robot_description/meshes/wheel_back_left.STL; visual mesh filename=package://robot_description/meshes/wheel_back_left.STL
- link wheel_back_right: geometry collision mesh filename=package://robot_description/meshes/wheel_back_right.STL; visual mesh filename=package://robot_description/meshes/wheel_back_right.STL
- link wheel_front_left: geometry collision mesh filename=package://robot_description/meshes/wheel_front_left.STL; visual mesh filename=package://robot_description/meshes/wheel_front_left.STL
- link wheel_front_right: geometry collision mesh filename=package://robot_description/meshes/wheel_front_right.STL; visual mesh filename=package://robot_description/meshes/wheel_front_right.STL
Joints:
- removed joint back_camera_dummy_joint
- removed joint front_camera_dummy_joint
- added joint back_camera_optical_joint: type fixed, parent back_camera, child back_camera_optical_frame, origin xyz=0 0 0 rpy=-1.5708 0 1.5708
- added joint front_camera_optical_joint: type fixed, parent front_camera, child front_camera_optical_frame, origin xyz=0 0 0 rpy=-1.5708 0 -1.5708
