Commit message: Nav2 intergration

File: src/robot_description/urdf/robot.urdf.xacro (robot description, xacro)
@@ -1,27 +1,4 @@
 <?xml version="1.0" ?>
 <robot name="cropMap_urdf" xmlns:xacro="http://www.ros.org/wiki/xacro">
-  <!-- Gazebo plugin includes -->
-  <gazebo>
-    <plugin name="gazebo_ros_control" filename="libgazebo_ros_control.so">
-      <robotNamespace>/cropMap_urdf</robotNamespace>
-      <robotSimType>gazebo_ros_control/DefaultRobotHWSim</robotSimType>
-    </plugin>
-  </gazebo>
-  <!-- Include Gazebo colors -->
-  <material name="dark_grey">
-    <color rgba="0.3 0.3 0.3 1.0"/>
-  </material>
-  <material name="light_grey">
-    <color rgba="0.79216 0.81961 0.93333 1"/>
-  </material>
-  <material name="blue">
-    <color rgba="0.0 0.0 0.8 1.0"/>
-  </material>
-  <material name="black">
-    <color rgba="0.0 0.0 0.0 1.0"/>
-  </material>
-  <material name="red">
-    <color rgba="1.0 0.0 0.0 1.0"/>
-  </material>
   <!-- Base Link -->
   <link name="base_link">
@@ -29,33 +6,28 @@
       <origin xyz="0.018582 -0.00058815 -0.099852" rpy="0 0 0" />
       <mass value="32.31" />
-      <inertia
-        ixx="0.92" ixy="0" ixz="0"
-        iyy="3.12" iyz="0"
-        izz="2.87" />
-    </inertial>
-    <visual>
-      <origin xyz="0 0 0" rpy="0 0 0" />
-      <geometry>
-        <mesh filename="file:///home/student/eiratech_ws/src/robot_description/meshes/base_link.STL" />
-      </geometry>
-      <material name="light_grey"/>
-    </visual>
-    <collision>
-      <origin xyz="0 0 0" rpy="0 0 0" />
-      <geometry>
-        <mesh filename="file:///home/student/eiratech_ws/src/robot_description/meshes/base_link.STL" />
-      </geometry>
-    </collision>
-  </link>
-  <!-- Gazebo material for base_link -->
-  <gazebo reference="base_link">
-    <material>Gazebo/Gray</material>
-  </gazebo>
-  <!-- Base footprint -->
+      <inertia ixx="0.92" ixy="0" ixz="0" iyy="3.12" iyz="0" izz="2.87" />
+    </inertial>
+    <visual>
+      <origin xyz="0 0 0" rpy="0 0 0" />
+      <geometry>
+        <mesh filename="file:///home/manish/eiratech_ws/install/robot_description/share/robot_description/meshes/base_link.STL" />
+      </geometry>
+      <material name="">
+        <color rgba="0.79216 0.81961 0.93333 1" />
+      </material>
+    </visual>
+    <collision>
+      <origin xyz="0 0 0" rpy="0 0 0" />
+      <geometry>
+	      <mesh filename="file:///home/manish/eiratech_ws/install/robot_description/share/robot_description/meshes/base_link.STL" />
+      </geometry>
+    </collision>
+  </link>
+  <!-- Base Footprint -->
   <link name="base_footprint"/>
   <joint name="base_footprint_ref_joint" type="fixed">
     <origin xyz="0 0 .25" rpy="0 0 0" />
     <parent link="base_footprint" />
-    <child link="base_link" />
+    <child link="base_link" />  <!-- Fixed typo: was "childggg" -->
     <axis xyz="0 1 0" />
   </joint>
@@ -64,21 +36,20 @@
     <inertial>
       <origin xyz="-3.8916E-11 0.012822 1.02E-07" rpy="0 0 0" />
-      <mass value=".041" />
-      <inertia
-        ixx="0.04" ixy="0.0" ixz="0.0"
-        iyy="0.05" iyz="0.0"
-        izz="0.04" />
-    </inertial>
-    <visual>
-      <origin xyz="0 0 0" rpy="0 0 0" />
-      <geometry>
-        <mesh filename="file:///home/student/eiratech_ws/src/robot_description/meshes/wheel_front_right.STL" />
-      </geometry>
-      <material name="light_grey"/>
-    </visual>
-    <collision>
-      <origin xyz="0 0 0" rpy="0 0 0" />
-      <geometry>
-        <mesh filename="file:///home/student/eiratech_ws/src/robot_description/meshes/wheel_front_right.STL" />
+      <mass value="2.5" />  <!-- Increased mass for better physics -->
+      <inertia ixx="0.04" ixy="0.0" ixz="0.0" iyy="0.05" iyz="0.0" izz="0.04" />
+    </inertial>
+    <visual>
+      <origin xyz="0 0 0" rpy="0 0 0" />
+      <geometry>
+        <mesh filename="file:///home/manish/eiratech_ws/install/robot_description/share/robot_description/meshes/wheel_front_right.STL" />
+      </geometry>
+      <material name="">
+        <color rgba="0.79216 0.81961 0.93333 1" />
+      </material>
+    </visual>
+    <collision>
+      <origin xyz="0 0 0" rpy="0 0 0" />
+      <geometry>
+        <mesh filename="file:///home/manish/eiratech_ws/install/robot_description/share/robot_description/meshes/wheel_front_right.STL" />
       </geometry>
     </collision>
@@ -89,38 +60,26 @@
     <child link="wheel_front_right" />
     <axis xyz="0 1 0" />
-    <dynamics damping="0.0001" friction="0.0001" />
-  </joint>
-  <!-- Gazebo plugin for front right wheel -->
-  <gazebo reference="wheel_front_right">
-    <material>Gazebo/DarkGray</material>
-    <mu1>1.0</mu1>
-    <mu2>1.0</mu2>
-    <kp>1000000.0</kp>
-    <kd>100.0</kd>
-    <minDepth>0.001</minDepth>
-    <maxVel>1.0</maxVel>
-    <fdir1>1 0 0</fdir1>
-  </gazebo>
+    <dynamics damping="0.1" friction="0.1" />
+  </joint>
   <!-- Back Right Wheel -->
   <link name="wheel_back_right">
     <inertial>
       <origin xyz="-3.8916E-11 0.012822 1.02E-07" rpy="0 0 0" />
-      <mass value=".041" />
-      <inertia
-        ixx="0.04" ixy="0.0" ixz="0.0"
-        iyy="0.05" iyz="0.0"
-        izz="0.04" />
-    </inertial>
-    <visual>
-      <origin xyz="0 0 0" rpy="0 0 0" />
-      <geometry>
-        <mesh filename="file:///home/student/eiratech_ws/src/robot_description/meshes/wheel_back_right.STL" />
-      </geometry>
-      <material name="light_grey"/>
-    </visual>
-    <collision>
-      <origin xyz="0 0 0" rpy="0 0 0" />
-      <geometry>
-        <mesh filename="file:///home/student/eiratech_ws/src/robot_description/meshes/wheel_back_right.STL" />
+      <mass value="2.5" />
+      <inertia ixx="0.04" ixy="0.0" ixz="0.0" iyy="0.05" iyz="0.0" izz="0.04" />
+    </inertial>
+    <visual>
+      <origin xyz="0 0 0" rpy="0 0 0" />
+      <geometry>
+        <mesh filename="file:///home/manish/eiratech_ws/install/robot_description/share/robot_description/meshes/wheel_back_right.STL" />
+      </geometry>
+      <material name="">
+        <color rgba="0.79216 0.81961 0.93333 1" />
+      </material>
+    </visual>
+    <collision>
+      <origin xyz="0 0 0" rpy="0 0 0" />
+      <geometry>
+	      <mesh filename="file:///home/manish/eiratech_ws/install/robot_description/share/robot_description/meshes/wheel_back_right.STL" />
       </geometry>
     </collision>
@@ -131,38 +90,26 @@
     <child link="wheel_back_right" />
     <axis xyz="0 1 0" />
-    <dynamics damping="0.0001" friction="0.0001" />
-  </joint>
-  <!-- Gazebo plugin for back right wheel -->
-  <gazebo reference="wheel_back_right">
-    <material>Gazebo/DarkGray</material>
-    <mu1>1.0</mu1>
-    <mu2>1.0</mu2>
-    <kp>1000000.0</kp>
-    <kd>100.0</kd>
-    <minDepth>0.001</minDepth>
-    <maxVel>1.0</maxVel>
-    <fdir1>1 0 0</fdir1>
-  </gazebo>
+    <dynamics damping="0.1" friction="0.1" />
+  </joint>
   <!-- Back Left Wheel -->
   <link name="wheel_back_left">
     <inertial>
       <origin xyz="-1.02E-07 -0.012822 3.8916E-11" rpy="0 0 0" />
-      <mass value=".041" />
-      <inertia
-        ixx="0.04" ixy="0.0" ixz="0.0"
-        iyy="0.05" iyz="0.0"
-        izz="0.04" />
-    </inertial>
-    <visual>
-      <origin xyz="0 0 0" rpy="0 0 0" />
-      <geometry>
-        <mesh filename="file:///home/student/eiratech_ws/src/robot_description/meshes/wheel_back_left.STL" />
-      </geometry>
-      <material name="light_grey"/>
-    </visual>
-    <collision>
-      <origin xyz="0 0 0" rpy="0 0 0" />
-      <geometry>
-        <mesh filename="file:///home/student/eiratech_ws/src/robot_description/meshes/wheel_back_left.STL" />
+      <mass value="2.5" />
+      <inertia ixx="0.04" ixy="0.0" ixz="0.0" iyy="0.05" iyz="0.0" izz="0.04" />
+    </inertial>
+    <visual>
+      <origin xyz="0 0 0" rpy="0 0 0" />
+      <geometry>
+        <mesh filename="file:///home/manish/eiratech_ws/install/robot_description/share/robot_description/meshes/wheel_back_left.STL" />
+      </geometry>
+      <material name="">
+        <color rgba="0.79216 0.81961 0.93333 1" />
+      </material>
+    </visual>
+    <collision>
+      <origin xyz="0 0 0" rpy="0 0 0" />
+      <geometry>
+        <mesh filename="file:///home/manish/eiratech_ws/install/robot_description/share/robot_description/meshes/wheel_back_left.STL" />
       </geometry>
     </collision>
@@ -173,38 +120,26 @@
     <child link="wheel_back_left" />
     <axis xyz="0 1 0" />
-    <dynamics damping="0.0001" friction="0.0001" />
-  </joint>
-  <!-- Gazebo plugin for back left wheel -->
-  <gazebo reference="wheel_back_left">
-    <material>Gazebo/DarkGray</material>
-    <mu1>1.0</mu1>
-    <mu2>1.0</mu2>
-    <kp>1000000.0</kp>
-    <kd>100.0</kd>
-    <minDepth>0.001</minDepth>
-    <maxVel>1.0</maxVel>
-    <fdir1>1 0 0</fdir1>
-  </gazebo>
+    <dynamics damping="0.1" friction="0.1" />
+  </joint>
   <!-- Front Left Wheel -->
   <link name="wheel_front_left">
     <inertial>
       <origin xyz="3.8916E-11 -0.012822 1.02E-07" rpy="0 0 0" />
-      <mass value=".041" />
-      <inertia
-        ixx="0.04" ixy="0.0" ixz="0.0"
-        iyy="0.05" iyz="0.0"
-        izz="0.04" />
-    </inertial>
-    <visual>
-      <origin xyz="0 0 0" rpy="0 0 0" />
-      <geometry>
-        <mesh filename="file:///home/student/eiratech_ws/src/robot_description/meshes/wheel_front_left.STL" />
-      </geometry>
-      <material name="light_grey"/>
-    </visual>
-    <collision>
-      <origin xyz="0 0 0" rpy="0 0 0" />
-      <geometry>
-        <mesh filename="file:///home/student/eiratech_ws/src/robot_description/meshes/wheel_front_left.STL" />
+      <mass value="2.5" />
+      <inertia ixx="0.04" ixy="0.0" ixz="0.0" iyy="0.05" iyz="0.0" izz="0.04" />
+    </inertial>
+    <visual>
+      <origin xyz="0 0 0" rpy="0 0 0" />
+      <geometry>
+        <mesh filename="file:///home/manish/eiratech_ws/install/robot_description/share/robot_description/meshes/wheel_front_left.STL" />
+      </geometry>
+      <material name="">
+        <color rgba="0.79216 0.81961 0.93333 1" />
+      </material>
+    </visual>
+    <collision>
+      <origin xyz="0 0 0" rpy="0 0 0" />
+      <geometry>
+        <mesh filename="file:///home/manish/eiratech_ws/install/robot_description/share/robot_description/meshes/wheel_front_left.STL" />
       </geometry>
     </collision>
@@ -215,33 +150,21 @@
     <child link="wheel_front_left" />
     <axis xyz="0 1 0" />
-    <dynamics damping="0.0001" friction="0.0001" />
-  </joint>
-  <!-- Gazebo plugin for front left wheel -->
-  <gazebo reference="wheel_front_left">
-    <material>Gazebo/DarkGray</material>
-    <mu1>1.0</mu1>
-    <mu2>1.0</mu2>
-    <kp>1000000.0</kp>
-    <kd>100.0</kd>
-    <minDepth>0.001</minDepth>
-    <maxVel>1.0</maxVel>
-    <fdir1>1 0 0</fdir1>
-  </gazebo>
+    <dynamics damping="0.1" friction="0.1" />
+  </joint>
   <!-- Back Camera -->
   <link name="back_camera">
     <inertial>
       <origin xyz="-0.032487 0.0089676 -0.0027971" rpy="0 0 0" />
-      <mass value="0.1" />
-      <inertia
-        ixx="0.001" ixy="0.0" ixz="0.0"
-        iyy="0.001" iyz="0.0"
-	      izz="0.001" />
-    </inertial>
-    <visual>
-      <origin xyz="0 0 0" rpy="0 0 0" />
-      <geometry>
-        <mesh filename="file:///home/student/eiratech_ws/src/robot_description/meshes/back_camera.STL" />
-      </geometry>
-      <material name="black"/>
+      <mass value="0.2" />  <!-- Added mass for physics -->
+      <inertia ixx="0.001" ixy="0.0" ixz="0.0" iyy="0.001" iyz="0.0" izz="0.001" />
+    </inertial>
+    <visual>
+      <origin xyz="0 0 0" rpy="0 0 0" />
+      <geometry>
+        <mesh filename="file:///home/manish/eiratech_ws/install/robot_description/share/robot_description/meshes/back_camera.STL" />
+      </geometry>
+      <material name="">
+        <color rgba="0.79216 0.81961 0.93333 1" />
+      </material>
     </visual>
   </link>
@@ -250,58 +173,21 @@
     <parent link="base_link" />
     <child link="back_camera" />
-  </joint>
-  <!-- Gazebo plugin for back camera -->
-  <gazebo reference="back_camera">
-    <sensor type="camera" name="back_camera">
-      <update_rate>30.0</update_rate>
-      <camera name="back">
-        <horizontal_fov>1.047</horizontal_fov>
-        <image>
-          <width>640</width>
-          <height>480</height>
-          <format>R8G8B8</format>
-        </image>
-        <clip>
-          <near>0.1</near>
-          <far>100</far>
-        </clip>
-        <noise>
-          <type>gaussian</type>
-          <mean>0.0</mean>
-          <stddev>0.007</stddev>
-        </noise>
-      </camera>
-      <plugin name="back_camera_controller" filename="libgazebo_ros_camera.so">
-        <alwaysOn>true</alwaysOn>
-        <updateRate>0.0</updateRate>
-        <cameraName>back_camera</cameraName>
-        <imageTopicName>image_raw</imageTopicName>
-        <cameraInfoTopicName>camera_info</cameraInfoTopicName>
-        <frameName>back_camera_optical_frame</frameName>
-        <hackBaseline>0.07</hackBaseline>
-        <distortionK1>0.0</distortionK1>
-        <distortionK2>0.0</distortionK2>
-        <distortionK3>0.0</distortionK3>
-        <distortionT1>0.0</distortionT1>
-        <distortionT2>0.0</distortionT2>
-      </plugin>
-    </sensor>
-  </gazebo>
+    <axis xyz="0 0 0" />
+  </joint>
   <!-- Front Camera -->
   <link name="front_camera">
     <inertial>
       <origin xyz="0.012395 -0.012586 0.0091516" rpy="0 0 0" />
-      <mass value="0.1" />
-      <inertia
-        ixx="0.001" ixy="0.0" ixz="0.0"
-        iyy="0.001" iyz="0.0"
-        izz="0.001" />
-    </inertial>
-    <visual>
-      <origin xyz="0 0 0" rpy="0 0 0" />
-      <geometry>
-        <mesh filename="file:///home/student/eiratech_ws/src/robot_description/meshes/front_camera.STL" />
-      </geometry>
-      <material name="black"/>
+      <mass value="0.2" />  <!-- Added mass for physics -->
+      <inertia ixx="0.001" ixy="0.0" ixz="0.0" iyy="0.001" iyz="0.0" izz="0.001" />
+    </inertial>
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